File: keypad/keypad.kicad_pcb (KiCad board)
At the start: 2 copper layers, 57.8 x 38.8 mm, 25 parts, among them J1 USB_C_Receptacle_USB2.0_14P, SW1 SW_Push, U1 STM32G031G8Ux, U2 USBLC6-2SC6, Y2 16MHz

Commit message: main
Parts:
- moved R1 25.7 mm to (123.3, 57.7), turned to 90 degrees
- moved C1 3.40 mm to (119.0, 48.5)
- moved C2 3.40 mm to (119.0, 53.9)
- moved Y2 3.40 mm to (118.9, 51.2)
Connections:
- U1 pad 12: unconnected-(U1-PA6-Pad12) -> Net-(MX3-COL)
- U1 pad 13: unconnected-(U1-PA7-Pad13) -> Net-(MX2-COL)
- U1 pad 19: unconnected-(U1-PA12/PA10-Pad19) -> Net-(D4-K)
- U1 pad 20: unconnected-(U1-PA13-Pad20) -> Net-(MX1-COL)
- U1 pad 21: unconnected-(U1-PA14-Pad21) -> Net-(D1-K)
Routing:
- net Net-(MX3-COL): track 19.0 -> 54.8 mm
- net +5V: track 72.9 -> 46.9 mm
- net Net-(D1-K): track 45.1 -> 64.2 mm, vias 0 -> 2
- net Net-(D4-K): track 43.7 -> 60.8 mm, vias 0 -> 2
- net Net-(MX2-COL): track 25.2 -> 41.4 mm
- net Net-(MX1-COL): track 24.0 -> 31.7 mm, vias 0 -> 1
- net GND: track 104.6 -> 101.2 mm, vias 4 -> 5
- net Net-(U1-PC14): track 8.68 -> 6.34 mm
- net Net-(U1-PC15): track 11.8 -> 9.57 mm
- net Net-(U1-PF2): track 49.2 -> 48.1 mm
