File: keypad/keypad.kicad_sch (KiCad schematic)
At the start: 7 parts, among them U1 STM32G031G8Ux

Commit message: main
Parts:
- added C1, C2: 22pF, symbol Device:C_Small
- added F1: Polyfuse_Small, symbol Device:Polyfuse_Small
- added J1: USB_C_Receptacle_USB2.0_14P, symbol Connector:USB_C_Receptacle_USB2.0_14P
- added MX1, MX2, MX3, MX4, MX5, MX6: MX-NoLED, symbol MX_Alps_Hybrid:MX-NoLED
- added R1: 10K, symbol Device:R_Small
- added R2, R3: 5K1, symbol Device:R_Small
- added R4, R5: 22, symbol Device:R_Small
- added SW1: SW_Push, symbol Switch:SW_Push
- added U2: USBLC6-2SC6, Package_TO_SOT_SMD:SOT-23-6, symbol Power_Protection:USBLC6-2SC6
- added Y1: 16MHz, symbol Device:Crystal_GND23_Small
Connections:
- net at D3.1 (K): now also D1.1 (K), D2.1 (K)
- net at D3.2 (A): now also MX3.2 (ROW)
- net at U1.1 (PC14): now also C1.2, Y1.1
- net at U1.2 (PC15): now also C2.2, Y1.4
- net at U1.26 (PB6): now also R5.2
- net at U1.27 (PB7): now also R4.2
- net at U1.5 (PF2): now also R1.2, SW1.2
- net at D2.2 (A): now also MX2.2 (ROW)
- net at D6.1 (K): now also D4.1 (K), D5.1 (K)
- net at D6.2 (A): now also MX6.2 (ROW)
- net at D4.2 (A): now also MX4.2 (ROW)
- net at D1.2 (A): now also MX1.2 (ROW)
- net at D5.2 (A): now also MX5.2 (ROW)
- new net: J1.A1 (GND), J1.A12 (GND), J1.B1 (GND), J1.B12 (GND), J1.S1 (SHIELD), U2.5 (VBUS)
- new net: F1.2, J1.A4 (VBUS), J1.A9 (VBUS), J1.B4 (VBUS), J1.B9 (VBUS)
- new net: J1.A5 (CC1), R2.2
- new net: J1.A6 (D+), J1.B6 (D+), U2.6 (I/O1)
- new net: J1.A7 (D-), J1.B7 (D-), U2.4 (I/O2)
- new net: J1.B5 (CC2), R3.2
- new net: MX1.1 (COL), MX4.1 (COL)
- new net: MX2.1 (COL), MX5.1 (COL)
- new net: MX3.1 (COL), MX6.1 (COL)
- new net: R4.1, U2.1 (I/O1)
- new net: R5.1, U2.3 (I/O2)
- new net +5V: F1.1, R1.1, U2.2 (GND)
- new net GND: C1.1, C2.1, R2.1, R3.1, SW1.1, Y1.2, Y1.3
Other:
- moved on the sheet: D1, D2, D3, D4, D5, D6, U1

Commit message: main
Parts:
- removed Y1: 16MHz, symbol Device:Crystal_GND23_Small
- added Y2: 16MHz, Crystal:Crystal_SMD_3225-4Pin_3.2x2.5mm, symbol Device:Crystal_GND24_Small
- C1, C2: footprint (none) -> Capacitor_SMD:C_0805_2012Metric
- F1: footprint (none) -> other_components:PF0805
- J1: footprint (none) -> Connector_USB:USB_C_Receptacle_GCT_USB4105-xx-A_16P_TopMnt_Horizontal
- MX1, MX2, MX3, MX4, MX5, MX6: footprint (none) -> Button_Switch_Keyboard:SW_Cherry_MX_1.00u_PCB
- R1, R2, R3, R4, R5: footprint (none) -> Resistor_SMD:R_0805_2012Metric
- SW1: footprint (none) -> Button_Switch_SMD:SW_Push_1P1T_NO_6x6mm_H9.5mm
Connections:
- net +5V: now also U1.4 (VSS)
- net GND: now also J1.A1 (GND), J1.A12 (GND), J1.B1 (GND), J1.B12 (GND), J1.S1 (SHIELD), U1.3 (VDD), U2.5 (VBUS), Y2.2, Y2.4
- net at C1.2, U1.1 (PC14): now also Y2.1
- net at C2.2, U1.2 (PC15): now also Y2.3
Other:
- moved on the sheet: D1, D2, D3, D4, D5, D6, MX1, MX2, MX3, MX4, MX5, MX6

Commit message: main
Connections:
- net at D1.1 (K), D2.1 (K), D3.1 (K): now also U1.21 (PA14)
- net at U1.12 (PA6): now also MX3.1 (COL), MX6.1 (COL)
- net at U1.13 (PA7): now also MX2.1 (COL), MX5.1 (COL)
- net at U1.19 (PA12/PA10): now also D4.1 (K), D5.1 (K), D6.1 (K)
- net at U1.20 (PA13): now also MX1.1 (COL), MX4.1 (COL)
Changed lines of the file:
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@@
+	)
+	(junction
+		(at 194.31 58.42)
+		(diameter 0)
+		(color 0 0 0 0)
 	)
 	(junction
@@
 	)
 	(junction
+		(at 168.91 74.93)
+		(diameter 0)
+		(color 0 0 0 0)
+	)
+	(junction
+		(at 184.15 53.34)
+		(diameter 0)
+		(color 0 0 0 0)
+	)
+	(junction
+		(at 168.91 50.8)
+		(diameter 0)
+		(color 0 0 0 0)
+	)
+	(junction
 		(at 101.6 101.6)
 		(diameter 0)
@@
 		(color 0 0 0 0)
 	)
+	(junction
+		(at 173.99 55.88)
+		(diameter 0)
+		(color 0 0 0 0)
+	)
 	(wire
 		(pts
@@
 	(wire
 		(pts
+			(xy 158.75 55.88) (xy 173.99 55.88)
+		)
+		(stroke
+			(width 0)
+			(type default)
+		)
+	)
+	(wire
+		(pts
 			(xy 104.14 25.4) (xy 104.14 27.94)
 		)
@@
 	(wire
 		(pts
+			(xy 156.21 58.42) (xy 156.21 74.93)
+		)
+		(stroke
+			(width 0)
+			(type default)
+		)
+	)
+	(wire
+		(pts
+			(xy 173.99 38.1) (xy 173.99 55.88)
+		)
+		(stroke
+			(width 0)
+			(type default)
+		)
+	)
+	(wire
+		(pts
 			(xy 83.82 44.45) (xy 88.9 44.45)
 		)
@@
 	(wire
 		(pts
+			(xy 163.83 48.26) (xy 163.83 58.42)
+		)
+		(stroke
+			(width 0)
+			(type default)
+		)
+	)
+	(wire
+		(pts
 			(xy 113.03 114.3) (xy 118.11 114.3)
 		)
@@
 	(wire
 		(pts
-			(xy 173.99 62.23) (xy 173.99 38.1)
+			(xy 146.05 63.5) (xy 140.97 63.5)
 		)
 		(stroke
@@
 	(wire
 		(pts
+			(xy 194.31 58.42) (xy 194.31 38.1)
+		)
+		(stroke
+			(width 0)
+			(type default)
+		)
+	)
+	(wire
+		(pts
 			(xy 90.17 63.5) (xy 105.41 63.5)
 		)
@@
 	(wire
 		(pts
+			(xy 143.51 50.8) (xy 143.51 53.34)
+		)
+		(stroke
+			(width 0)
+			(type default)
+		)
+	)
+	(wire
+		(pts
 			(xy 179.07 74.93) (xy 168.91 74.93)
 		)
@@
 	(wire
 		(pts
+			(xy 140.97 50.8) (xy 143.51 50.8)
+		)
+		(stroke
+			(width 0)
+			(type default)
+		)
+	)
+	(wire
+		(pts
 			(xy 107.95 106.68) (xy 118.11 106.68)
 		)
@@
 	(wire
 		(pts
+			(xy 173.99 55.88) (xy 173.99 62.23)
+		)
+		(stroke
+			(width 0)
+			(type default)
+		)
+	)
+	(wire
+		(pts
+			(xy 143.51 53.34) (xy 184.15 53.34)
+		)
+		(stroke
+			(width 0)
+			(type default)
+		)
+	)
+	(wire
+		(pts
 			(xy 87.63 60.96) (xy 96.52 60.96)
 		)
@@
 	(wire
 		(pts
+			(xy 140.97 58.42) (xy 156.21 58.42)
+		)
+		(stroke
+			(width 0)
+			(type default)
+		)
+	)
+	(wire
+		(pts
 			(xy 73.66 33.02) (xy 73.66 39.37)
 		)
@@
 	(wire
 		(pts
-			(xy 194.31 62.23) (xy 194.31 38.1)
+			(xy 158.75 60.96) (xy 158.75 55.88)
+		)
+		(stroke
+			(width 0)
+			(type default)
+		)
+	)
+	(wire
+		(pts
+			(xy 194.31 62.23) (xy 194.31 58.42)
 		)
 		(stroke
@@
 	(wire
 		(pts
+			(xy 168.91 50.8) (xy 179.07 50.8)
+		)
+		(stroke
+			(width 0)
+			(type default)
+		)
+	)
+	(wire
+		(pts
 			(xy 73.66 44.45) (xy 73.66 48.26)
 		)
@@
 	(wire
 		(pts
+			(xy 146.05 50.8) (xy 168.91 50.8)
+		)
+		(stroke
+			(width 0)
+			(type default)
+		)
+	)
+	(wire
+		(pts
 			(xy 113.03 100.33) (xy 118.11 100.33)
 		)
@@
 	(wire
 		(pts
+			(xy 163.83 58.42) (xy 194.31 58.42)
+		)
+		(stroke
+			(width 0)
+			(type default)
+		)
+	)
+	(wire
+		(pts
+			(xy 156.21 74.93) (xy 168.91 74.93)
+		)
+		(stroke
+			(width 0)
+			(type default)
+		)
+	)
+	(wire
+		(pts
 			(xy 128.27 22.86) (xy 123.19 22.86)
 		)
@@
 	(wire
 		(pts
-			(xy 184.15 62.23) (xy 184.15 38.1)
+			(xy 184.15 62.23) (xy 184.15 53.34)
 		)
 		(stroke
@@
 	(wire
 		(pts
+			(xy 146.05 50.8) (xy 146.05 63.5)
+		)
+		(stroke
+			(width 0)
+			(type default)
+		)
+	)
+	(wire
+		(pts
 			(xy 83.82 39.37) (xy 88.9 39.37)
 		)
@@
 	(wire
 		(pts
+			(xy 140.97 60.96) (xy 158.75 60.96)
+		)
+		(stroke
+			(width 0)
+			(type default)
+		)
+	)
+	(wire
+		(pts
+			(xy 140.97 48.26) (xy 163.83 48.26)
+		)
+		(stroke
+			(width 0)
+			(type default)
+		)
+	)
+	(wire
+		(pts
 			(xy 87.63 86.36) (xy 90.17 86.36)
 		)
@@
 	(wire
 		(pts
-			(xy 179.07 50.8) (xy 168.91 50.8)
-		)
-		(stroke
+			(xy 184.15 53.34) (xy 184.15 38.1)
+		)
+		(stroke
